Commit message: Set limit for testing

File: robots/lumyai_neli.URDF (robot description, URDF)
Before this commit: robot lumyai_neli, 21 links, 20 joints
Joints:
- joint right_elbow_joint: limit (none) -> lower=-1.6 upper=0 effort=30 velocity=0.4; type continuous -> revolute
- joint right_shoulder_1_joint: limit (none) -> lower=0 upper=2.35525 effort=30 velocity=0.4; type continuous -> revolute

Commit message: Fix direction of tilt_joint

File: robots/lumyai_neli.URDF (robot description, URDF)
Before this commit: robot lumyai_neli, 21 links, 20 joints
Joints:
- joint right_elbow_joint: axis 0 1 0 -> 0 -1 0; limit lower=-1.6 upper=0 effort=30 velocity=0.4 -> lower=0 upper=2.5 effort=30 velocity=0.4
- joint right_shoulder_1_joint: limit lower=0 upper=2.35525 effort=30 velocity=0.4 -> lower=-0.5 upper=2.35525 effort=30 velocity=0.4
- joint tilt_joint: axis 0 1 0 -> 0 -1 0

Commit message: update URDF

File: robots/lumyai_neli.URDF (robot description, URDF)
Before this commit: robot lumyai_neli, 21 links, 20 joints
Joints:
- joint right_shoulder_2_joint: axis 1 0 0 -> -1 0 0

Commit message: Add camera_link and camera_joint

File: robots/lumyai_neli.URDF (robot description, URDF)
Before this commit: robot lumyai_neli, 21 links, 20 joints
Links:
- added link camera_link
Joints:
- added joint camera_joint: type fixed, parent tilt_Link, child camera_link, origin xyz=0.02832 -0.0606 0.04405 rpy=0 0 0, axis 0 0 1

Commit message: Change initial value of torso_link(prismatic)

File: robots/lumyai_neli.URDF (robot description, URDF)
Before this commit: robot lumyai_neli, 22 links, 21 joints
Joints:
- joint right_shoulder_2_joint: limit (none) -> lower=-1.57 upper=1.57 effort=30 velocity=0.4; type continuous -> revolute
- joint right_wrist_1_joint: limit (none) -> lower=-0.7 upper=3.14 effort=30 velocity=0.4; type continuous -> revolute
- joint torso_joint: origin xyz=0.075 0 0.5342 rpy=-1.2246E-16 -1.2246E-16 -4.1633E-17 -> xyz=0.075 0 0.34 rpy=-1.2246E-16 -1.2246E-16 -4.1633E-17

Commit message: Reconfig axis for right shoulder & right elbow

File: robots/lumyai_neli.URDF (robot description, URDF)
Before this commit: robot lumyai_neli, 22 links, 21 joints
Joints:
- joint left_elbow_joint: origin xyz=0.278 0 0 rpy=1.3878E-16 -1.1102E-16 0 -> xyz=0.278 0 0 rpy=1.3878E-16 -1.57075 0
- joint left_shoulder_1_joint: origin xyz=-0.025 0.0858 0.485 rpy=5.593E-17 3.6739E-16 -8.1621E-17 -> xyz=-0.025 0.0858 0.485 rpy=5.593E-17 1.57075 -8.1621E-17
- joint right_elbow_joint: limit lower=0 upper=2.5 effort=30 velocity=0.4 -> lower=-1.7 upper=1.0 effort=30 velocity=0.4; origin xyz=0.278 0 0 rpy=-1.6008E-15 -1.2246E-16 1.6653E-16 -> xyz=0.278 0 0 rpy=-1.6008E-15 -1.57075 1.6653E-16
- joint right_shoulder_1_joint: limit lower=-0.5 upper=2.35525 effort=30 velocity=0.4 -> lower=-1.7 upper=0.8 effort=30 velocity=0.4; origin xyz=-0.025 -0.0828 0.485 rpy=5.9764E-17 1.2246E-16 1.0433E-16 -> xyz=-0.025 -0.0828 0.485 rpy=5.9764E-17 1.57075 1.0433E-16

Commit message: Set limit of gripper

File: robots/lumyai_neli.URDF (robot description, URDF)
Before this commit: robot lumyai_neli, 22 links, 21 joints
Joints:
- joint right_gripper_joint: limit (none) -> lower=-1.0 upper=0.0 effort=30 velocity=0.4; type continuous -> revolute

Commit message: update URDF wrist 1 2 3 joint limit

File: robots/lumyai_neli.URDF (robot description, URDF)
Before this commit: robot lumyai_neli, 22 links, 21 joints
Joints:
- joint right_wrist_2_joint: limit (none) -> lower=-0.47 upper=1.57 effort=30 velocity=0.4; type continuous -> revolute
- joint right_wrist_3_joint: limit (none) -> lower=-1.57 upper=1.57 effort=30 velocity=0.4; type continuous -> revolute

Commit message: update URDF

File: robots/lumyai_neli.URDF (robot description, URDF)
Before this commit: robot lumyai_neli, 22 links, 21 joints
Joints:
- joint right_gripper_joint: limit lower=-1.0 upper=0.0 effort=30 velocity=0.4 -> lower=-0.8 upper=0.0 effort=30 velocity=0.4
- joint right_wrist_1_joint: limit lower=-0.7 upper=3.14 effort=30 velocity=0.4 -> lower=-0.7 upper=3.04 effort=30 velocity=0.4
- joint right_wrist_2_joint: limit lower=-0.47 upper=1.57 effort=30 velocity=0.4 -> lower=-0.5 upper=1.31 effort=30 velocity=0.4

Commit message: update URDF

File: robots/lumyai_neli.URDF (robot description, URDF)
Before this commit: robot lumyai_neli, 22 links, 21 joints
Joints:
- joint right_shoulder_1_joint: limit lower=-1.7 upper=0.8 effort=30 velocity=0.4 -> lower=-1.82 upper=0.59 effort=30 velocity=0.4

Commit message: re-calib again

File: robots/lumyai_neli.URDF (robot description, URDF)
Before this commit: robot lumyai_neli, 22 links, 21 joints
Joints:
- joint right_wrist_2_joint: limit lower=-0.5 upper=1.31 effort=30 velocity=0.4 -> lower=-0.5 upper=1.45 effort=30 velocity=0.4

Commit message: add leftarm

File: robots/lumyai_neli.URDF (robot description, URDF)
Before this commit: robot lumyai_neli, 22 links, 21 joints
Joints:
- joint left_shoulder_1_joint: axis 0 1 0 -> 0 -1 0
- joint left_shoulder_2_joint: axis 1 0 0 -> -1 0 0
- joint right_elbow_joint: limit lower=-1.7 upper=1.0 effort=30 velocity=0.4 -> lower=-1.7 upper=0.2 effort=30 velocity=0.4
- joint right_wrist_2_joint: limit lower=-0.5 upper=1.45 effort=30 velocity=0.4 -> lower=-1.40 upper=1.45 effort=30 velocity=0.4

Commit message: leftwrist: config revolute

File: robots/lumyai_neli.URDF (robot description, URDF)
Before this commit: robot lumyai_neli, 22 links, 21 joints
Joints:
- joint left_wrist_1_joint: limit (none) -> lower=-0.7 upper=3.04 effort=30 velocity=0.4; type continuous -> revolute
- joint left_wrist_2_joint: limit (none) -> lower=-0.6 upper=1.60 effort=30 velocity=0.4; type continuous -> revolute
- joint left_wrist_3_joint: limit (none) -> lower=-1.57 upper=1.57 effort=30 velocity=0.4; type continuous -> revolute
- joint right_wrist_2_joint: limit lower=-1.40 upper=1.45 effort=30 velocity=0.4 -> lower=-1.40 upper=1.60 effort=30 velocity=0.4

Commit message: update URDF

File: robots/lumyai_neli.URDF (robot description, URDF)
Before this commit: robot lumyai_neli, 22 links, 21 joints
Joints:
- joint right_wrist_2_joint: limit lower=-1.40 upper=1.60 effort=30 velocity=0.4 -> lower=-0.5 upper=1.60 effort=30 velocity=0.4

Commit message: after robocup2015

File: robots/lumyai_neli.URDF (robot description, URDF)
Before this commit: robot lumyai_neli, 22 links, 21 joints
Joints:
- joint right_wrist_2_joint: limit lower=-0.5 upper=1.60 effort=30 velocity=0.4 -> lower=-0.5 upper=1.90 effort=30 velocity=0.4

Commit message: adjust URDF to the new calib

File: robots/lumyai_neli.URDF (robot description, URDF)
Before this commit: robot lumyai_neli, 22 links, 21 joints
Joints:
- joint right_gripper_joint: limit lower=-0.8 upper=0.0 effort=30 velocity=0.4 -> lower=-0.74 upper=0.0 effort=30 velocity=0.4
- joint right_wrist_2_joint: limit lower=-0.5 upper=1.90 effort=30 velocity=0.4 -> lower=-0.5 upper=1.60 effort=30 velocity=0.4

Commit message: update bound URDF

File: robots/lumyai_neli.URDF (robot description, URDF)
Before this commit: robot lumyai_neli, 22 links, 21 joints
Joints:
- joint right_elbow_joint: limit lower=-1.7 upper=0.2 effort=30 velocity=0.4 -> lower=-1.0 upper=0.22 effort=30 velocity=0.4
- joint right_gripper_joint: limit lower=-0.74 upper=0.0 effort=30 velocity=0.4 -> lower=-0.8 upper=1.1 effort=30 velocity=0.4
- joint right_shoulder_1_joint: limit lower=-1.82 upper=0.59 effort=30 velocity=0.4 -> lower=-1.2 upper=0.5 effort=30 velocity=0.4
- joint right_shoulder_2_joint: limit lower=-1.57 upper=1.57 effort=30 velocity=0.4 -> lower=-1.47 upper=1.1 effort=30 velocity=0.4
- joint right_wrist_1_joint: limit lower=-0.7 upper=3.04 effort=30 velocity=0.4 -> lower=-3.1 upper=2.5 effort=30 velocity=0.4
- joint right_wrist_2_joint: limit lower=-0.5 upper=1.60 effort=30 velocity=0.4 -> lower=-0.6 upper=1.5 effort=30 velocity=0.4
- joint right_wrist_3_joint: limit lower=-1.57 upper=1.57 effort=30 velocity=0.4 -> lower=-2.64 upper=3.17 effort=30 velocity=0.4

Commit message: Adding Link for Inverse Kinemetic

File: robots/lumyai_neli.URDF (robot description, URDF)
Before this commit: robot lumyai_neli, 22 links, 21 joints
Links:
- added link left_mani_link
- added link right_mani_link
Joints:
- added joint left_mani_joint: type fixed, parent torso_Link, child left_mani_link, origin xyz=-0.025 0.17 0.486 rpy=0 0 0, axis 0 0 1
- added joint right_mani_joint: type fixed, parent torso_Link, child right_mani_link, origin xyz=-0.025 -0.17 0.486 rpy=0 0 0, axis 0 0 1

Commit message: edit bound right arm

File: robots/lumyai_neli.URDF (robot description, URDF)
Before this commit: robot lumyai_neli, 24 links, 23 joints
Joints:
- joint left_elbow_joint: limit (none) -> lower=-0.889 upper=0.17 effort=30 velocity=0.4; type continuous -> revolute
- joint left_mani_joint: origin xyz=-0.025 0.17 0.486 rpy=0 0 0 -> xyz=-0.02 0.17 0.8 rpy=0 0 0
- joint left_shoulder_1_joint: axis 0 -1 0 -> 0 1 0; limit (none) -> lower=-1.2 upper=0.589 effort=30 velocity=0.4; type continuous -> revolute
- joint left_shoulder_2_joint: limit (none) -> lower=-1.5 upper=1.0 effort=30 velocity=0.4; type continuous -> revolute
- joint left_wrist_1_joint: limit lower=-0.7 upper=3.04 effort=30 velocity=0.4 -> lower=-3.1 upper=2.5 effort=30 velocity=0.4
- joint left_wrist_2_joint: limit lower=-0.6 upper=1.60 effort=30 velocity=0.4 -> lower=-0.6 upper=1.50 effort=30 velocity=0.4
- joint left_wrist_3_joint: limit lower=-1.57 upper=1.57 effort=30 velocity=0.4 -> lower=-2.64 upper=3.17 effort=30 velocity=0.4
- joint right_elbow_joint: axis 0 -1 0 -> 0 1 0
- joint right_gripper_fixed_joint: limit (none) -> lower=-0.8 upper=0.2 effort=30 velocity=0.4; type fixed -> revolute
- joint right_gripper_joint: limit lower=-0.8 upper=1.1 effort=30 velocity=0.4 -> lower=-0.8 upper=0.2 effort=30 velocity=0.4
- joint right_mani_joint: origin xyz=-0.025 -0.17 0.486 rpy=0 0 0 -> xyz=-0.02 -0.17 0.8 rpy=0 0 0
- joint right_shoulder_1_joint: axis 0 1 0 -> 0 -1 0; limit lower=-1.2 upper=0.5 effort=30 velocity=0.4 -> lower=-0.3 upper=1.3 effort=30 velocity=0.4
- joint right_shoulder_2_joint: axis -1 0 0 -> 1 0 0; limit lower=-1.47 upper=1.1 effort=30 velocity=0.4 -> lower=-0.8 upper=1.6 effort=30 velocity=0.4

Commit message: edit URDF

File: robots/lumyai_neli.URDF (robot description, URDF)
Before this commit: robot lumyai_neli, 24 links, 23 joints
Joints:
- joint right_elbow_joint: limit lower=-1.0 upper=0.22 effort=30 velocity=0.4 -> lower=-0.3 upper=1.0 effort=30 velocity=0.4

Commit message: update URDF

File: robots/lumyai_neli.URDF (robot description, URDF)
Before this commit: robot lumyai_neli, 24 links, 23 joints
Joints:
- joint right_elbow_joint: axis 0 1 0 -> 0 -1 0; limit lower=-0.3 upper=1.0 effort=30 velocity=0.4 -> lower=-1.0 upper=0.22 effort=30 velocity=0.4
- joint right_gripper_joint: limit lower=-0.8 upper=0.2 effort=30 velocity=0.4 -> lower=0.0 upper=0.8 effort=30 velocity=0.4
- joint right_shoulder_1_joint: axis 0 -1 0 -> 0 1 0; limit lower=-0.3 upper=1.3 effort=30 velocity=0.4 -> lower=-1.2 upper=0.5 effort=30 velocity=0.4
- joint right_shoulder_2_joint: axis 1 0 0 -> -1 0 0; limit lower=-0.8 upper=1.6 effort=30 velocity=0.4 -> lower=-1.47 upper=1.1 effort=30 velocity=0.4

Commit message: add right/left mani link

File: robots/lumyai_neli.URDF (robot description, URDF)
Before this commit: robot lumyai_neli, 24 links, 23 joints
Joints:
- joint left_mani_joint: origin xyz=-0.02 0.17 0.8 rpy=0 0 0 -> xyz=-0.025 0.17 0.486 rpy=0 0 0
- joint right_elbow_joint: limit lower=-1.0 upper=0.22 effort=30 velocity=0.4 -> lower=-1.5 upper=0.22 effort=30 velocity=0.4
- joint right_mani_joint: origin xyz=-0.02 -0.17 0.8 rpy=0 0 0 -> xyz=-0.025 -0.17 0.486 rpy=0 0 0
- joint right_shoulder_1_joint: limit lower=-1.2 upper=0.5 effort=30 velocity=0.4 -> lower=-1.9 upper=0.5 effort=30 velocity=0.4

Commit message: backup from ketamine

File: robots/lumyai_neli.URDF (robot description, URDF)
Before this commit: robot lumyai_neli, 24 links, 23 joints
Joints:
- joint right_elbow_joint: limit lower=-1.5 upper=0.22 effort=30 velocity=0.4 -> lower=-1.0 upper=0.22 effort=30 velocity=0.4
- joint right_shoulder_1_joint: limit lower=-1.9 upper=0.5 effort=30 velocity=0.4 -> lower=-1.2 upper=0.5 effort=30 velocity=0.4

Commit message: update update bound limit

File: robots/lumyai_neli.URDF (robot description, URDF)
Before this commit: robot lumyai_neli, 24 links, 23 joints
Joints:
- joint right_elbow_joint: limit lower=-1.0 upper=0.22 effort=30 velocity=0.4 -> lower=-1.5 upper=0.22 effort=30 velocity=0.4
- joint right_shoulder_1_joint: limit lower=-1.2 upper=0.5 effort=30 velocity=0.4 -> lower=-1.35 upper=0.4 effort=30 velocity=0.4

Commit message: update urdf

File: robots/lumyai_neli.URDF (robot description, URDF)
Before this commit: robot lumyai_neli, 24 links, 23 joints
Joints:
- joint right_shoulder_1_joint: limit lower=-1.35 upper=0.4 effort=30 velocity=0.4 -> lower=-1.5 upper=0.4 effort=30 velocity=0.4

Commit message: Add damping factor for simulation

File: robots/lumyai_neli.URDF (robot description, URDF)
Before this commit: robot lumyai_neli, 24 links, 23 joints
Joints:
- joint right_gripper_fixed_joint: limit lower=-0.8 upper=0.2 effort=30 velocity=0.4 -> (none); type revolute -> fixed

Commit message: Set all mass about zero to avoid inertia and make robot fall

File: robots/lumyai_neli.URDF (robot description, URDF)
Before this commit: robot lumyai_neli, 24 links, 23 joints
Links:
- link base_link: mass 22.8330889899799 -> 42.8330889899799
- link laser_Link: mass 0.229160254925421 -> 0.001
- link left_elbow_Link: mass 0.166643682967829 -> 0.001
- link left_gripper_Link: mass 0.0226554217932752 -> 0.001
- link left_gripper_fixed_Link: mass 0.0226554217932752 -> 0.001
- link left_shoulder_1_Link: mass 0.489568995899366 -> 0.001
- link left_shoulder_2_Link: mass 0.232391134105839 -> 0.001
- link left_wrist_1_Link: mass 0.0149816280592893 -> 0.001
- link left_wrist_2_Link: mass 0.0641453083227973 -> 0.001
- link left_wrist_3_Link: mass 0.0557526551260178 -> 0.001
- link pan_Link: mass 0.0300690193079437 -> 0.001
- link right_elbow_Link: mass 0.166643682967829 -> 0.001
- link right_gripper_Link: mass 0.0226554217932752 -> 0.001
- link right_gripper_fixed_Link: mass 0.0226554217932752 -> 0.001
- link right_shoulder_1_Link: mass 0.489568995899366 -> 0.001
- link right_shoulder_2_Link: mass 0.232391134105839 -> 0.001
- link right_wrist_1_Link: mass 0.0149816280592893 -> 0.001
- link right_wrist_2_Link: mass 0.0641453083227973 -> 0.001
- link right_wrist_3_Link: mass 0.0557526551260179 -> 0.001
- link tilt_Link: mass 0.833552168165174 -> 0.001
- link torso_Link: mass 2.69155190066383 -> 0.001

Commit message: update config

File: robots/lumyai_neli.URDF (robot description, URDF)
Before this commit: robot lumyai_neli, 24 links, 23 joints
Joints:
- joint left_elbow_joint: axis 0 1 0 -> 0 -1 0
- joint left_shoulder_1_joint: axis 0 1 0 -> 0 -1 0

Commit message: update init torso_Link

File: robots/lumyai_neli.URDF (robot description, URDF)
Before this commit: robot lumyai_neli, 24 links, 23 joints
Joints:
- joint left_elbow_joint: limit lower=-0.889 upper=0.17 effort=30 velocity=0.4 -> lower=-1.502134 upper=0.402 effort=30 velocity=0.4
- joint left_shoulder_1_joint: limit lower=-1.2 upper=0.589 effort=30 velocity=0.4 -> lower=-0.506337 upper=1.3625 effort=30 velocity=0.4
- joint left_shoulder_2_joint: limit lower=-1.5 upper=1.0 effort=30 velocity=0.4 -> lower=-1.4515 upper=1.67552 effort=30 velocity=0.4
- joint left_wrist_1_joint: limit lower=-3.1 upper=2.5 effort=30 velocity=0.4 -> lower=-2.5 upper=3.1 effort=30 velocity=0.4
- joint left_wrist_2_joint: limit lower=-0.6 upper=1.50 effort=30 velocity=0.4 -> lower=-0.6 upper=1.5 effort=30 velocity=0.4
- joint torso_joint: origin xyz=0.075 0 0.34 rpy=-1.2246E-16 -1.2246E-16 -4.1633E-17 -> xyz=0.075 0 0.305 rpy=-1.2246E-16 -1.2246E-16 -4.1633E-17

Commit message: update lumyai_neli.URDF

File: robots/lumyai_neli.URDF (robot description, URDF)
Before this commit: robot lumyai_neli, 24 links, 23 joints
Joints:
- joint left_gripper_joint: axis 0 0 1 -> 0 0 -1; limit (none) -> lower=0.0 upper=0.8 effort=30 velocity=0.4; type continuous -> revolute
- joint left_wrist_2_joint: limit lower=-0.6 upper=1.5 effort=30 velocity=0.4 -> lower=-0.6 upper=1.75 effort=30 velocity=0.4
- joint right_shoulder_1_joint: axis 0 1 0 -> 0 -1 0; limit lower=-1.5 upper=0.4 effort=30 velocity=0.4 -> lower=-0.4 upper=1.5 effort=30 velocity=0.4
- joint torso_joint: limit lower=0 upper=0 effort=0 velocity=0 -> lower=0 upper=0.24 effort=30 velocity=0.4

Commit message: add lumyai_neli.URDF

File: robots/lumyai_neli.URDF (robot description, URDF)
Before this commit: robot lumyai_neli, 24 links, 23 joints
Links:
- added link base_footprint
- added link imu_link
Joints:
- added joint base_footprint_joint: type fixed, parent base_link, child base_footprint, origin xyz=0 0 0 rpy=0 0 0, axis 0 0 1
- added joint imu_joint: type fixed, parent base_link, child imu_link, origin xyz=0.252 0 0.1492 rpy=0 0 0, axis 0 0 1

Commit message: Update lumyai_neli.URDF

File: robots/lumyai_neli.URDF (robot description, URDF)
Before this commit: robot lumyai_neli, 26 links, 25 joints
Joints:
- joint imu_joint: origin xyz=0.252 0 0.1492 rpy=0 0 0 -> xyz=0.122 -0.16 0.1492 rpy=0 0 3.1416

Commit message: Update lumyai_neli.URDF

File: robots/lumyai_neli.URDF (robot description, URDF)
Before this commit: robot lumyai_neli, 26 links, 25 joints
Joints:
- joint imu_joint: origin xyz=0.122 -0.16 0.1492 rpy=0 0 3.1416 -> xyz=0.122 -0.015 0.1492 rpy=3.1416 0 0

Commit message: edit imu rpy

File: robots/lumyai_neli.URDF (robot description, URDF)
Before this commit: robot lumyai_neli, 26 links, 25 joints
Links:
- removed link base_footprint
Joints:
- removed joint base_footprint_joint
- joint imu_joint: origin xyz=0.122 -0.015 0.1492 rpy=3.1416 0 0 -> xyz=0.122 -0.000 0.1492 rpy=0 0 0
